File: hackpad/hackpad.kicad_pcb (KiCad board)
At the start: 2 copper layers, 112 x 105 mm, 36 parts, among them SW1 SW_Push_45deg, SW10 SW_Push_45deg, SW11 SW_Push_45deg, SW13 SW_Push_45deg, SW14 SW_Push_45deg, SW15 SW_Push_45deg, SW16 SW_Push_45deg, SW17 SW_Push_45deg, SW19 SW_Push_45deg, SW2 SW_Push_45deg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

Commit message: more hackpad stuff! woo!
Parts:
- added REF**: MountingHole_3.2mm_M3, MountingHole:MountingHole_3.2mm_M3, F.Cu at (224.5, 120.0)
- added REF**: MountingHole_3.2mm_M3, MountingHole:MountingHole_3.2mm_M3, F.Cu at (125.5, 119.5)
- added REF**: MountingHole_3.2mm_M3, MountingHole:MountingHole_3.2mm_M3, F.Cu at (216.0, 61.5)
- added REF**: MountingHole_3.2mm_M3, MountingHole:MountingHole_3.2mm_M3, F.Cu at (123.5, 43.0)
Routing:
- net Net-(U1-GPIO2/SCK): track 212.9 -> 212.3 mm
Other:
- outline, holes or cut-outs redrawn

Commit message: add all the files, start with firmware
Parts:
- removed D14: D, Diode_THT:D_DO-35_SOD27_P7.62mm_Horizontal
- removed SW19: SW_Push_45deg, hackpad:SW_Cherry_MX_1.00u_PCB
Routing:
- net Net-(D14-A): track 13.3 -> 0.00 mm
- net Net-(D5-K): track 153.5 -> 153.3 mm, vias 2 -> 3
