File: hackpad/hackpad.kicad_sch (KiCad schematic)
At the start: 35 parts, among them SW1 SW_Push_45deg, SW10 SW_Push_45deg, SW11 SW_Push_45deg, SW13 SW_Push_45deg, SW14 SW_Push_45deg, SW15 SW_Push_45deg, SW16 SW_Push_45deg, SW17 SW_Push_45deg, SW19 SW_Push_45deg, SW2 SW_Push_45deg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

Commit message: more hackpad stuff! woo!
Parts:
- SW1, SW10, SW11, SW13, SW14, SW15, SW19, SW2, SW3, SW4, SW5, SW6, SW7, SW9: footprint Button_Switch_Keyboard:SW_Cherry_MX_1.00u_PCB -> hackpad:SW_Cherry_MX_1.00u_PCB
- SW16, SW8: footprint Button_Switch_Keyboard:SW_Cherry_MX_2.00u_Vertical_PCB -> hackpad:SW_Cherry_MX_2.00u_Vertical_PCB
- SW17: footprint Button_Switch_Keyboard:SW_Cherry_MX_2.00u_PCB -> hackpad:SW_Cherry_MX_2.00u_PCB
- U1: footprint OPL:XIAO-RP2040-SMD -> hackpad:XIAO-RP2040-DIP
Changed lines of the file:
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@@
 			)
 		)
-		(property "Footprint" "Button_Switch_Keyboard:SW_Cherry_MX_1.00u_PCB"
+		(property "Footprint" "hackpad:SW_Cherry_MX_1.00u_PCB"
 			(at 62.23 86.36 0)
 			(effects
@@
 			)
 		)
-		(property "Footprint" "Button_Switch_Keyboard:SW_Cherry_MX_1.00u_PCB"
+		(property "Footprint" "hackpad:SW_Cherry_MX_1.00u_PCB"
 			(at 46.99 55.88 0)
 			(effects
@@
 			)
 		)
-		(property "Footprint" "Button_Switch_Keyboard:SW_Cherry_MX_1.00u_PCB"
+		(property "Footprint" "hackpad:SW_Cherry_MX_1.00u_PCB"
 			(at 62.23 55.88 0)
 			(effects
@@
 			)
 		)
-		(property "Footprint" "Button_Switch_Keyboard:SW_Cherry_MX_1.00u_PCB"
+		(property "Footprint" "hackpad:SW_Cherry_MX_1.00u_PCB"
 			(at 46.99 86.36 0)
 			(effects
@@
 			)
 		)
-		(property "Footprint" "Button_Switch_Keyboard:SW_Cherry_MX_1.00u_PCB"
+		(property "Footprint" "hackpad:SW_Cherry_MX_1.00u_PCB"
 			(at 31.75 71.12 0)
 			(effects
@@
 			)
 		)
-		(property "Footprint" "OPL:XIAO-RP2040-SMD"
+		(property "Footprint" "hackpad:XIAO-RP2040-DIP"
 			(at 128.778 86.868 0)
 			(effects
@@
 			)
 		)
-		(property "Footprint" "Button_Switch_Keyboard:SW_Cherry_MX_1.00u_PCB"
+		(property "Footprint" "hackpad:SW_Cherry_MX_1.00u_PCB"
 			(at 46.99 101.6 0)
 			(effects
@@
 			)
 		)
-		(property "Footprint" "Button_Switch_Keyboard:SW_Cherry_MX_1.00u_PCB"
+		(property "Footprint" "hackpad:SW_Cherry_MX_1.00u_PCB"
 			(at 31.75 55.88 0)
 			(effects
@@
 			)
 		)
-		(property "Footprint" "Button_Switch_Keyboard:SW_Cherry_MX_1.00u_PCB"
+		(property "Footprint" "hackpad:SW_Cherry_MX_1.00u_PCB"
 			(at 62.23 101.6 0)
 			(effects
@@
 			)
 		)
-		(property "Footprint" "Button_Switch_Keyboard:SW_Cherry_MX_1.00u_PCB"
+		(property "Footprint" "hackpad:SW_Cherry_MX_1.00u_PCB"
 			(at 31.75 101.6 0)
 			(effects
@@
 			)
 		)
-		(property "Footprint" "Button_Switch_Keyboard:SW_Cherry_MX_2.00u_Vertical_PCB"
+		(property "Footprint" "hackpad:SW_Cherry_MX_2.00u_Vertical_PCB"
 			(at 77.47 101.6 0)
 			(effects
@@
 			)
 		)
-		(property "Footprint" "Button_Switch_Keyboard:SW_Cherry_MX_2.00u_PCB"
+		(property "Footprint" "hackpad:SW_Cherry_MX_2.00u_PCB"
 			(at 31.75 116.84 0)
 			(effects
@@
 			)
 		)
-		(property "Footprint" "Button_Switch_Keyboard:SW_Cherry_MX_1.00u_PCB"
+		(property "Footprint" "hackpad:SW_Cherry_MX_1.00u_PCB"
 			(at 62.23 116.84 0)
 			(effects
@@
 			)
 		)
-		(property "Footprint" "Button_Switch_Keyboard:SW_Cherry_MX_2.00u_Vertical_PCB"
+		(property "Footprint" "hackpad:SW_Cherry_MX_2.00u_Vertical_PCB"
 			(at 77.47 71.12 0)
 			(effects
@@
 			)
 		)
-		(property "Footprint" "Button_Switch_Keyboard:SW_Cherry_MX_1.00u_PCB"
+		(property "Footprint" "hackpad:SW_Cherry_MX_1.00u_PCB"
 			(at 46.99 71.12 0)
 			(effects
@@
 			)
 		)
-		(property "Footprint" "Button_Switch_Keyboard:SW_Cherry_MX_1.00u_PCB"
+		(property "Footprint" "hackpad:SW_Cherry_MX_1.00u_PCB"
 			(at 62.23 71.12 0)
 			(effects
@@
 			)
 		)
-		(property "Footprint" "Button_Switch_Keyboard:SW_Cherry_MX_1.00u_PCB"
+		(property "Footprint" "hackpad:SW_Cherry_MX_1.00u_PCB"
 			(at 31.75 86.36 0)
 			(effects
@@
 			)
 		)
-		(property "Footprint" "Button_Switch_Keyboard:SW_Cherry_MX_1.00u_PCB"
+		(property "Footprint" "hackpad:SW_Cherry_MX_1.00u_PCB"
 			(at 77.47 55.88 0)
 			(effects

Commit message: add all the files, start with firmware
Parts:
- removed D14: D, Diode_THT:D_DO-35_SOD27_P7.62mm_Horizontal, symbol Device:D
- removed SW19: SW_Push_45deg, hackpad:SW_Cherry_MX_1.00u_PCB, symbol Switch:SW_Push_45deg
Changed lines of the file:
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@@
-	)
-	(junction
-		(at 59.69 114.3)
-		(diameter 0)
-		(color 0 0 0 0)
 	)
 	(junction
@@
 	)
 	(junction
-		(at 64.77 127)
-		(diameter 0)
-		(color 0 0 0 0)
-	)
-	(junction
 		(at 49.53 111.76)
 		(diameter 0)
@@
 	(wire
 		(pts
-			(xy 59.69 99.06) (xy 59.69 114.3)
+			(xy 59.69 99.06) (xy 59.69 128.27)
 		)
 		(stroke
@@
 	(wire
 		(pts
-			(xy 64.77 127) (xy 109.22 127)
+			(xy 34.29 127) (xy 109.22 127)
 		)
 		(stroke
@@
 	(wire
 		(pts
-			(xy 34.29 127) (xy 64.77 127)
-		)
-		(stroke
-			(width 0)
-			(type default)
-		)
-	)
-	(wire
-		(pts
 			(xy 29.21 114.3) (xy 29.21 133.35)
 		)
@@
 		(pts
 			(xy 34.29 96.52) (xy 49.53 96.52)
-		)
-		(stroke
-			(width 0)
-			(type default)
-		)
-	)
-	(wire
-		(pts
-			(xy 59.69 114.3) (xy 59.69 128.27)
 		)
 		(stroke
@@
 	(symbol
 		(lib_id "Device:D")
-		(at 64.77 123.19 90)
-		(unit 1)
-		(exclude_from_sim no)
-		(in_bom yes)
-		(on_board yes)
-		(dnp no)
-		(fields_autoplaced yes)
-		(property "Reference" "D14"
-			(at 67.31 121.9199 90)
-			(effects
-				(font
-					(size 1.27 1.27)
-				)
-				(justify right)
-			)
-		)
-		(property "Value" "D"
-			(at 67.31 124.4599 90)
-			(effects
-				(font
-					(size 1.27 1.27)
-				)
-				(justify right)
-			)
-		)
-		(property "Footprint" "Diode_THT:D_DO-35_SOD27_P7.62mm_Horizontal"
-			(at 64.77 123.19 0)
-			(effects
-				(font
-					(size 1.27 1.27)
-				)
-				(hide yes)
-			)
-		)
-		(property "Datasheet" "~"
-			(at 64.77 123.19 0)
-			(effects
-				(font
-					(size 1.27 1.27)
-				)
-				(hide yes)
-			)
-		)
-		(property "Description" "Diode"
-			(at 64.77 123.19 0)
-			(effects
-				(font
-					(size 1.27 1.27)
-				)
-				(hide yes)
-			)
-		)
-		(property "Sim.Device" "D"
-			(at 64.77 123.19 0)
-			(effects
-				(font
-					(size 1.27 1.27)
-				)
-				(hide yes)
-			)
-		)
-		(property "Sim.Pins" "1=K 2=A"
-			(at 64.77 123.19 0)
-			(effects
-				(font
-					(size 1.27 1.27)
-				)
-				(hide yes)
-			)
-		)
-		(pin "1"
-		)
-		(pin "2"
-		)
-		(instances
-			(project ""
-				(path "/e13dbd81-e82e-4825-a082-450068fce1d9"
-					(reference "D14")
-					(unit 1)
-				)
-			)
-		)
-	)
-	(symbol
-		(lib_id "Device:D")
 		(at 49.53 107.95 90)
 		(unit 1)
@@
 					(unit 1)
 				)
-			)
-		)
-	)
-	(symbol
-		(lib_id "Switch:SW_Push_45deg")
-		(at 62.23 116.84 0)
-		(unit 1)
-		(exclude_from_sim no)
-		(in_bom yes)
-		(on_board yes)
-		(dnp no)
-		(fields_autoplaced yes)
-		(property "Reference" "SW19"
-			(at 62.23 109.22 0)
-			(effects
-				(font
-					(size 1.27 1.27)
-				)
-			)
-		)
-		(property "Value" "SW_Push_45deg"
-			(at 62.23 111.76 0)
-			(effects
-				(font
-					(size 1.27 1.27)
-				)
-			)
-		)
-		(property "Footprint" "hackpad:SW_Cherry_MX_1.00u_PCB"
-			(at 62.23 116.84 0)
-			(effects
-				(font
-					(size 1.27 1.27)
-				)
-				(hide yes)
-			)
-		)
-		(property "Datasheet" "~"
-			(at 62.23 116.84 0)
-			(effects
-				(font
-					(size 1.27 1.27)
-				)
-				(hide yes)
-			)
-		)
-		(property "Description" "Push button switch, normally open, two pins, 45° tilted"
-			(at 62.23 116.84 0)
-			(effects
-				(font
-					(size 1.27 1.27)
-				)
-				(hide yes)
-			)
-		)
-		(pin "1"
-		)
-		(pin "2"
-		)
-		(instances
-			(project "Untitled"
-				(path "/e13dbd81-e82e-4825-a082-450068fce1d9"
-					(reference "SW19")
-					(unit 1)
-				)
